File: hardware/lightstick.sch (EAGLE design)
At the start: 0 parts

Commit message: added connector for 12V power supply
Parts:
- added X1, X2: RIA182-02, con-ria182:RIA182-02
Connections:
- new net +12V: X1-1.SK, X2-1.SK
- new net GND: X1-2.SK, X2-2.SK
Other:
- note added: "power supply"
Changed lines of the file:
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@@
 <setting verticaltext="up"/>
 </settings>
-<grid distance="0.1" unitdist="inch" unit="inch" style="lines" multiple="1" display="no" altdistance="0.01" altunitdist="inch" altunit="inch"/>
+<grid distance="0.1" unitdist="inch" unit="mm" style="lines" multiple="1" display="yes" altdistance="0.01" altunitdist="inch" altunit="mm"/>
 <layers>
 <layer number="1" name="Top" color="4" fill="1" visible="no" active="no"/>
@@
 <parts>
 <part name="FRAME1" library="frames" deviceset="A4L-LOC" device=""/>
+<part name="X1" library="con-ria182" deviceset="RIA182-02" device=""/>
+<part name="X2" library="con-ria182" deviceset="RIA182-02" device=""/>
+<part name="P+1" library="supply1" deviceset="+12V" device=""/>
+<part name="P+2" library="supply1" deviceset="+12V" device=""/>
+<part name="GND1" library="supply1" deviceset="GND" device=""/>
+<part name="GND2" library="supply1" deviceset="GND" device=""/>
 </parts>
 <sheets>
 <sheet>
 <plain>
+<text x="10.16" y="43.18" size="1.778" layer="91">power supply</text>
 </plain>
 <instances>
 <instance part="FRAME1" gate="G$1" x="0" y="0"/>
+<instance part="X1" gate="-1" x="22.86" y="27.94"/>
+<instance part="X1" gate="-2" x="22.86" y="22.86"/>
+<instance part="X2" gate="-1" x="48.26" y="27.94"/>
+<instance part="X2" gate="-2" x="48.26" y="22.86"/>
+<instance part="P+1" gate="1" x="30.48" y="35.56"/>
+<instance part="P+2" gate="1" x="55.88" y="35.56"/>
+<instance part="GND1" gate="1" x="30.48" y="15.24"/>
+<instance part="GND2" gate="1" x="55.88" y="15.24"/>
 </instances>
 <busses>
 </busses>
 <nets>
+<net name="GND" class="0">
+<segment>
+<pinref part="X1" gate="-2" pin="SK"/>
+<pinref part="GND1" gate="1" pin="GND"/>
+<wire x1="27.94" y1="22.86" x2="30.48" y2="22.86" width="0.1524" layer="91"/>
+<wire x1="30.48" y1="22.86" x2="30.48" y2="17.78" width="0.1524" layer="91"/>
+</segment>
+<segment>
+<pinref part="X2" gate="-2" pin="SK"/>
+<pinref part="GND2" gate="1" pin="GND"/>
+<wire x1="53.34" y1="22.86" x2="55.88" y2="22.86" width="0.1524" layer="91"/>
+<wire x1="55.88" y1="22.86" x2="55.88" y2="17.78" width="0.1524" layer="91"/>
+</segment>
+</net>
+<net name="+12V" class="0">
+<segment>
+<pinref part="X1" gate="-1" pin="SK"/>
+<pinref part="P+1" gate="1" pin="+12V"/>
+<wire x1="27.94" y1="27.94" x2="30.48" y2="27.94" width="0.1524" layer="91"/>
+<wire x1="30.48" y1="27.94" x2="30.48" y2="33.02" width="0.1524" layer="91"/>
+</segment>
+<segment>
+<pinref part="X2" gate="-1" pin="SK"/>
+<pinref part="P+2" gate="1" pin="+12V"/>
+<wire x1="53.34" y1="27.94" x2="55.88" y2="27.94" width="0.1524" layer="91"/>
+<wire x1="55.88" y1="27.94" x2="55.88" y2="33.02" width="0.1524" layer="91"/>
+</segment>
+</net>
 </nets>
 </sheet>

Commit message: added connector for LED stripe
Parts:
- added JP1: (no value), pinhead:PINHD-1X3
Connections:
- new net +5V: JP1.1
- new net DATA: JP1.2
- net GND: now also JP1.3
Other:
- note added: "to LED stripe"
Changed lines of the file:
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@@
 <part name="GND1" library="supply1" deviceset="GND" device=""/>
 <part name="GND2" library="supply1" deviceset="GND" device=""/>
+<part name="JP1" library="pinhead" deviceset="PINHD-1X3" device=""/>
+<part name="P+3" library="supply1" deviceset="+5V" device=""/>
+<part name="GND3" library="supply1" deviceset="GND" device=""/>
 </parts>
 <sheets>
@@
 <plain>
 <text x="10.16" y="43.18" size="1.778" layer="91">power supply</text>
+<text x="106.68" y="35.56" size="1.778" layer="91">to LED stripe</text>
 </plain>
 <instances>
@@
 <instance part="GND1" gate="1" x="30.48" y="15.24"/>
 <instance part="GND2" gate="1" x="55.88" y="15.24"/>
+<instance part="JP1" gate="A" x="124.46" y="25.4"/>
+<instance part="P+3" gate="1" x="111.76" y="33.02"/>
+<instance part="GND3" gate="1" x="111.76" y="17.78"/>
 </instances>
 <busses>
@@
 <wire x1="55.88" y1="22.86" x2="55.88" y2="17.78" width="0.1524" layer="91"/>
 </segment>
+<segment>
+<pinref part="JP1" gate="A" pin="3"/>
+<pinref part="GND3" gate="1" pin="GND"/>
+<wire x1="121.92" y1="22.86" x2="111.76" y2="22.86" width="0.1524" layer="91"/>
+<wire x1="111.76" y1="22.86" x2="111.76" y2="20.32" width="0.1524" layer="91"/>
+</segment>
 </net>
 <net name="+12V" class="0">
@@
 </segment>
 </net>
+<net name="+5V" class="0">
+<segment>
+<pinref part="JP1" gate="A" pin="1"/>
+<pinref part="P+3" gate="1" pin="+5V"/>
+<wire x1="121.92" y1="27.94" x2="111.76" y2="27.94" width="0.1524" layer="91"/>
+<wire x1="111.76" y1="27.94" x2="111.76" y2="30.48" width="0.1524" layer="91"/>
+</segment>
+</net>
+<net name="DATA" class="0">
+<segment>
+<pinref part="JP1" gate="A" pin="2"/>
+<wire x1="121.92" y1="25.4" x2="111.76" y2="25.4" width="0.1524" layer="91"/>
+<label x="111.76" y="25.4" size="1.778" layer="95" rot="R180" xref="yes"/>
+</segment>
+</net>

Commit message: added switch for programming mode
Parts:
- added JP2: (no value), pinhead:PINHD-1X3
Connections:
- net DATA renamed DATA/GPIO2
- new net GPIO0: JP2.2
- net +5V: now also JP2.1
- net GND: now also JP2.3
Other:
- note added: "for programming: connect GPIO0 to +3V3 for normal operation: connect GPIO to GND"
- note added: "programming switch"
Changed lines of the file:
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@@
 <part name="P+3" library="supply1" deviceset="+5V" device=""/>
 <part name="GND3" library="supply1" deviceset="GND" device=""/>
+<part name="JP2" library="pinhead" deviceset="PINHD-1X3" device=""/>
+<part name="P+4" library="supply1" deviceset="+3V3" device=""/>
+<part name="GND4" library="supply1" deviceset="GND" device=""/>
 </parts>
 <sheets>
@@
 <text x="10.16" y="43.18" size="1.778" layer="91">power supply</text>
 <text x="106.68" y="35.56" size="1.778" layer="91">to LED stripe</text>
+<text x="152.4" y="68.58" size="1.778" layer="91">programming switch</text>
+<text x="144.78" y="40.64" size="1.778" layer="91">for programming: connect GPIO0 to +3V3
+for normal operation: connect GPIO to GND</text>
 </plain>
 <instances>
@@
 <instance part="P+3" gate="1" x="111.76" y="33.02"/>
 <instance part="GND3" gate="1" x="111.76" y="17.78"/>
+<instance part="JP2" gate="A" x="170.18" y="58.42"/>
+<instance part="P+4" gate="G$1" x="157.48" y="66.04"/>
+<instance part="GND4" gate="1" x="157.48" y="50.8"/>
 </instances>
 <busses>
@@
 <wire x1="111.76" y1="22.86" x2="111.76" y2="20.32" width="0.1524" layer="91"/>
 </segment>
+<segment>
+<pinref part="JP2" gate="A" pin="3"/>
+<pinref part="GND4" gate="1" pin="GND"/>
+<wire x1="167.64" y1="55.88" x2="157.48" y2="55.88" width="0.1524" layer="91"/>
+<wire x1="157.48" y1="55.88" x2="157.48" y2="53.34" width="0.1524" layer="91"/>
+</segment>
 </net>
 <net name="+12V" class="0">
@@
 <wire x1="111.76" y1="27.94" x2="111.76" y2="30.48" width="0.1524" layer="91"/>
 </segment>
+<segment>
+<pinref part="JP2" gate="A" pin="1"/>
+<pinref part="P+4" gate="G$1" pin="+3V3"/>
+<wire x1="167.64" y1="60.96" x2="157.48" y2="60.96" width="0.1524" layer="91"/>
+<wire x1="157.48" y1="60.96" x2="157.48" y2="63.5" width="0.1524" layer="91"/>
+</segment>
 </net>
-<net name="DATA" class="0">
+<net name="DATA/GPIO2" class="0">
 <segment>
 <pinref part="JP1" gate="A" pin="2"/>
 <wire x1="121.92" y1="25.4" x2="111.76" y2="25.4" width="0.1524" layer="91"/>
 <label x="111.76" y="25.4" size="1.778" layer="95" rot="R180" xref="yes"/>
+</segment>
+</net>
+<net name="GPIO0" class="0">
+<segment>
+<pinref part="JP2" gate="A" pin="2"/>
+<wire x1="167.64" y1="58.42" x2="157.48" y2="58.42" width="0.1524" layer="91"/>
+<label x="157.48" y="58.42" size="1.778" layer="95" rot="R180" xref="yes"/>
 </segment>
 </net>
@@
 </schematic>
 </drawing>
+<compatibility>
+<note version="6.3" minversion="6.2.2" severity="warning">
+Since Version 6.2.2 text objects can contain more than one line,
+which will not be processed correctly with this version.
+</note>
+</compatibility>
 </eagle>

Commit message: added UART connector
Parts:
- added JP3: (no value), pinhead:PINHD-1X3
Connections:
- new net RX: JP3.1
- new net TX: JP3.2
- net GND: now also JP3.3
Other:
- note added: "UART"
- moved on the sheet: JP2
Changed lines of the file:
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@@
 <part name="P+4" library="supply1" deviceset="+3V3" device=""/>
 <part name="GND4" library="supply1" deviceset="GND" device=""/>
+<part name="JP3" library="pinhead" deviceset="PINHD-1X3" device=""/>
+<part name="GND5" library="supply1" deviceset="GND" device=""/>
 </parts>
 <sheets>
@@
 <text x="10.16" y="43.18" size="1.778" layer="91">power supply</text>
 <text x="106.68" y="35.56" size="1.778" layer="91">to LED stripe</text>
-<text x="152.4" y="68.58" size="1.778" layer="91">programming switch</text>
-<text x="144.78" y="40.64" size="1.778" layer="91">for programming: connect GPIO0 to +3V3
+<text x="17.78" y="83.82" size="1.778" layer="91">programming switch</text>
+<text x="10.16" y="55.88" size="1.778" layer="91">for programming: connect GPIO0 to +3V3
 for normal operation: connect GPIO to GND</text>
+<text x="12.7" y="119.38" size="1.778" layer="91">UART</text>
 </plain>
 <instances>
@@
 <instance part="P+3" gate="1" x="111.76" y="33.02"/>
 <instance part="GND3" gate="1" x="111.76" y="17.78"/>
-<instance part="JP2" gate="A" x="170.18" y="58.42"/>
-<instance part="P+4" gate="G$1" x="157.48" y="66.04"/>
-<instance part="GND4" gate="1" x="157.48" y="50.8"/>
+<instance part="JP2" gate="A" x="35.56" y="73.66"/>
+<instance part="P+4" gate="G$1" x="22.86" y="81.28"/>
+<instance part="GND4" gate="1" x="22.86" y="66.04"/>
+<instance part="JP3" gate="A" x="30.48" y="109.22"/>
+<instance part="GND5" gate="1" x="17.78" y="101.6"/>
 </instances>
 <busses>
@@
 <pinref part="JP2" gate="A" pin="3"/>
 <pinref part="GND4" gate="1" pin="GND"/>
-<wire x1="167.64" y1="55.88" x2="157.48" y2="55.88" width="0.1524" layer="91"/>
-<wire x1="157.48" y1="55.88" x2="157.48" y2="53.34" width="0.1524" layer="91"/>
+<wire x1="33.02" y1="71.12" x2="22.86" y2="71.12" width="0.1524" layer="91"/>
+<wire x1="22.86" y1="71.12" x2="22.86" y2="68.58" width="0.1524" layer="91"/>
+</segment>
+<segment>
+<pinref part="JP3" gate="A" pin="3"/>
+<pinref part="GND5" gate="1" pin="GND"/>
+<wire x1="27.94" y1="106.68" x2="17.78" y2="106.68" width="0.1524" layer="91"/>
+<wire x1="17.78" y1="106.68" x2="17.78" y2="104.14" width="0.1524" layer="91"/>
 </segment>
 </net>
@@
 <pinref part="JP2" gate="A" pin="1"/>
 <pinref part="P+4" gate="G$1" pin="+3V3"/>
-<wire x1="167.64" y1="60.96" x2="157.48" y2="60.96" width="0.1524" layer="91"/>
-<wire x1="157.48" y1="60.96" x2="157.48" y2="63.5" width="0.1524" layer="91"/>
+<wire x1="33.02" y1="76.2" x2="22.86" y2="76.2" width="0.1524" layer="91"/>
+<wire x1="22.86" y1="76.2" x2="22.86" y2="78.74" width="0.1524" layer="91"/>
 </segment>
 </net>
@@
 <pinref part="JP1" gate="A" pin="2"/>
 <wire x1="121.92" y1="25.4" x2="111.76" y2="25.4" width="0.1524" layer="91"/>
-<label x="111.76" y="25.4" size="1.778" layer="95" rot="R180" xref="yes"/>
+<label x="111.76" y="25.4" size="1.27" layer="95" rot="R180" xref="yes"/>
 </segment>
 </net>
@@
 <segment>
 <pinref part="JP2" gate="A" pin="2"/>
-<wire x1="167.64" y1="58.42" x2="157.48" y2="58.42" width="0.1524" layer="91"/>
-<label x="157.48" y="58.42" size="1.778" layer="95" rot="R180" xref="yes"/>
+<wire x1="33.02" y1="73.66" x2="22.86" y2="73.66" width="0.1524" layer="91"/>
+<label x="22.86" y="73.66" size="1.27" layer="95" rot="R180" xref="yes"/>
 </segment>
 </net>
+<net name="RX" class="0">
+<segment>
+<pinref part="JP3" gate="A" pin="1"/>
+<wire x1="27.94" y1="111.76" x2="17.78" y2="111.76" width="0.1524" layer="91"/>
+<label x="17.78" y="111.76" size="1.27" layer="95" rot="R180" xref="yes"/>
+</segment>
+</net>
+<net name="TX" class="0">
+<segment>
+<pinref part="JP3" gate="A" pin="2"/>
+<wire x1="27.94" y1="109.22" x2="17.78" y2="109.22" width="0.1524" layer="91"/>
+<label x="17.78" y="109.22" size="1.27" layer="95" rot="R180" xref="yes"/>
+</segment>
+</net>

Commit message: added voltage regulator for 3V3
Parts:
- added C1, C2: 1u, rcl:C-EUC0805
- added U1: MCP1703AT-3302E/CB, lightstick:MCP1703AT-3302E/CB
Connections:
- new net +3V3: C2.1, U1.VOUT
- net +5V: now also C1.1, U1.VIN
- net GND: now also C1.2, C2.2, U1.GND
Other:
- note added: "Voltage regulator 5V -> 3V3"
Changed lines of the file:
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@@
 <part name="JP3" library="pinhead" deviceset="PINHD-1X3" device=""/>
 <part name="GND5" library="supply1" deviceset="GND" device=""/>
+<part name="U1" library="lightstick" deviceset="MCP1703AT-3302E/CB" device=""/>
+<part name="P+5" library="supply1" deviceset="+5V" device=""/>
+<part name="+3V1" library="supply1" deviceset="+3V3" device=""/>
+<part name="GND6" library="supply1" deviceset="GND" device=""/>
+<part name="C1" library="rcl" deviceset="C-EU" device="C0805" value="1u"/>
+<part name="C2" library="rcl" deviceset="C-EU" device="C0805" value="1u"/>
+<part name="GND7" library="supply1" deviceset="GND" device=""/>
+<part name="GND8" library="supply1" deviceset="GND" device=""/>
 </parts>
 <sheets>
@@
 for normal operation: connect GPIO to GND</text>
 <text x="12.7" y="119.38" size="1.778" layer="91">UART</text>
+<text x="193.04" y="167.64" size="1.27" layer="91">Voltage regulator 5V -&gt; 3V3</text>
 </plain>
 <instances>
@@
 <instance part="JP3" gate="A" x="30.48" y="109.22"/>
 <instance part="GND5" gate="1" x="17.78" y="101.6"/>
+<instance part="U1" gate="A" x="213.36" y="154.94"/>
+<instance part="P+5" gate="1" x="185.42" y="162.56"/>
+<instance part="+3V1" gate="G$1" x="241.3" y="162.56"/>
+<instance part="GND6" gate="1" x="193.04" y="142.24"/>
+<instance part="C1" gate="G$1" x="185.42" y="152.4"/>
+<instance part="C2" gate="G$1" x="241.3" y="152.4"/>
+<instance part="GND7" gate="1" x="185.42" y="142.24"/>
+<instance part="GND8" gate="1" x="241.3" y="142.24"/>
 </instances>
 <busses>
@@
 <wire x1="17.78" y1="106.68" x2="17.78" y2="104.14" width="0.1524" layer="91"/>
 </segment>
+<segment>
+<pinref part="C1" gate="G$1" pin="2"/>
+<pinref part="GND7" gate="1" pin="GND"/>
+<wire x1="185.42" y1="147.32" x2="185.42" y2="144.78" width="0.1524" layer="91"/>
+</segment>
+<segment>
+<pinref part="U1" gate="A" pin="GND"/>
+<wire x1="195.58" y1="149.86" x2="193.04" y2="149.86" width="0.1524" layer="91"/>
+<pinref part="GND6" gate="1" pin="GND"/>
+<wire x1="193.04" y1="149.86" x2="193.04" y2="144.78" width="0.1524" layer="91"/>
+</segment>
+<segment>
+<pinref part="C2" gate="G$1" pin="2"/>
+<pinref part="GND8" gate="1" pin="GND"/>
+<wire x1="241.3" y1="147.32" x2="241.3" y2="144.78" width="0.1524" layer="91"/>
+</segment>
 </net>
 <net name="+12V" class="0">
@@
 <wire x1="33.02" y1="76.2" x2="22.86" y2="76.2" width="0.1524" layer="91"/>
 <wire x1="22.86" y1="76.2" x2="22.86" y2="78.74" width="0.1524" layer="91"/>
+</segment>
+<segment>
+<pinref part="P+5" gate="1" pin="+5V"/>
+<pinref part="C1" gate="G$1" pin="1"/>
+<wire x1="185.42" y1="160.02" x2="185.42" y2="154.94" width="0.1524" layer="91"/>
+<pinref part="U1" gate="A" pin="VIN"/>
+<wire x1="195.58" y1="154.94" x2="185.42" y2="154.94" width="0.1524" layer="91"/>
+<junction x="185.42" y="154.94"/>
 </segment>
 </net>
@@
 </segment>
 </net>
+<net name="+3V3" class="0">
+<segment>
+<pinref part="C2" gate="G$1" pin="1"/>
+<pinref part="+3V1" gate="G$1" pin="+3V3"/>
+<wire x1="241.3" y1="154.94" x2="241.3" y2="160.02" width="0.1524" layer="91"/>
+<pinref part="U1" gate="A" pin="VOUT"/>
+<wire x1="231.14" y1="154.94" x2="241.3" y2="154.94" width="0.1524" layer="91"/>
+<junction x="241.3" y="154.94"/>
+</segment>
+</net>

Commit message: corrected comment regarding programming switch
Other:
- note added: "for programming: connect GPIO0 to GND for normal operation: connect GPIO to +3V3"
- note removed: "for programming: connect GPIO0 to +3V3 for normal operation: connect GPIO to GND"
Changed lines of the file:
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@@
 <text x="106.68" y="35.56" size="1.778" layer="91">to LED stripe</text>
 <text x="17.78" y="83.82" size="1.778" layer="91">programming switch</text>
-<text x="10.16" y="55.88" size="1.778" layer="91">for programming: connect GPIO0 to +3V3
-for normal operation: connect GPIO to GND</text>
+<text x="10.16" y="55.88" size="1.778" layer="91">for programming: connect GPIO0 to GND
+for normal operation: connect GPIO to +3V3</text>
 <text x="12.7" y="119.38" size="1.778" layer="91">UART</text>
 <text x="193.04" y="167.64" size="1.27" layer="91">Voltage regulator 5V -&gt; 3V3</text>

Commit message: added ESP 8266 controller
Parts:
- added U$1: ESP8266, lightstick:ESP8266
Connections:
- removed net DATA/GPIO2: JP1.2
- removed net GPIO0: JP2.2
- new net DATA: JP1.2, U$1.DATA/GPIO2
- new net PROGRAM: JP2.2, U$1.GPIO0
- net +3V3: now also U$1.CH_PD, U$1.RST, U$1.VCC
- net GND: now also U$1.GND
- net RX: now also U$1.RX
- net TX: now also U$1.TX
Other:
- note added: "ESP 8266 controller"
Changed lines of the file:
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@@
 <part name="GND7" library="supply1" deviceset="GND" device=""/>
 <part name="GND8" library="supply1" deviceset="GND" device=""/>
+<part name="U$1" library="lightstick" deviceset="ESP8266" device=""/>
+<part name="P+6" library="supply1" deviceset="+3V3" device=""/>
+<part name="GND9" library="supply1" deviceset="GND" device=""/>
 </parts>
 <sheets>
@@
 <text x="12.7" y="119.38" size="1.778" layer="91">UART</text>
 <text x="193.04" y="167.64" size="1.27" layer="91">Voltage regulator 5V -&gt; 3V3</text>
+<text x="86.36" y="104.14" size="1.27" layer="91">ESP 8266 controller</text>
 </plain>
 <instances>
@@
 <instance part="GND7" gate="1" x="185.42" y="142.24"/>
 <instance part="GND8" gate="1" x="241.3" y="142.24"/>
+<instance part="U$1" gate="A" x="111.76" y="83.82"/>
+<instance part="P+6" gate="G$1" x="86.36" y="99.06"/>
+<instance part="GND9" gate="1" x="86.36" y="68.58"/>
 </instances>
 <busses>
@@
 <pinref part="GND8" gate="1" pin="GND"/>
 <wire x1="241.3" y1="147.32" x2="241.3" y2="144.78" width="0.1524" layer="91"/>
+</segment>
+<segment>
+<pinref part="U$1" gate="A" pin="GND"/>
+<pinref part="GND9" gate="1" pin="GND"/>
+<wire x1="93.98" y1="76.2" x2="86.36" y2="76.2" width="0.1524" layer="91"/>
+<wire x1="86.36" y1="76.2" x2="86.36" y2="71.12" width="0.1524" layer="91"/>
 </segment>
 </net>
@@
 </segment>
 </net>
-<net name="DATA/GPIO2" class="0">
-<segment>
-<pinref part="JP1" gate="A" pin="2"/>
-<wire x1="121.92" y1="25.4" x2="111.76" y2="25.4" width="0.1524" layer="91"/>
-<label x="111.76" y="25.4" size="1.27" layer="95" rot="R180" xref="yes"/>
-</segment>
-</net>
-<net name="GPIO0" class="0">
-<segment>
-<pinref part="JP2" gate="A" pin="2"/>
-<wire x1="33.02" y1="73.66" x2="22.86" y2="73.66" width="0.1524" layer="91"/>
-<label x="22.86" y="73.66" size="1.27" layer="95" rot="R180" xref="yes"/>
-</segment>
-</net>
 <net name="RX" class="0">
 <segment>
@@
 <label x="17.78" y="111.76" size="1.27" layer="95" rot="R180" xref="yes"/>
 </segment>
+<segment>
+<pinref part="U$1" gate="A" pin="RX"/>
+<wire x1="129.54" y1="91.44" x2="137.16" y2="91.44" width="0.1524" layer="91"/>
+<label x="137.16" y="91.44" size="1.27" layer="95" xref="yes"/>
+</segment>
 </net>
 <net name="TX" class="0">
@@
 <wire x1="27.94" y1="109.22" x2="17.78" y2="109.22" width="0.1524" layer="91"/>
 <label x="17.78" y="109.22" size="1.27" layer="95" rot="R180" xref="yes"/>
+</segment>
+<segment>
+<pinref part="U$1" gate="A" pin="TX"/>
+<wire x1="129.54" y1="86.36" x2="137.16" y2="86.36" width="0.1524" layer="91"/>
+<label x="137.16" y="86.36" size="1.27" layer="95" xref="yes"/>
 </segment>
 </net>
@@
 <junction x="241.3" y="154.94"/>
 </segment>
-</net>
+<segment>
+<pinref part="U$1" gate="A" pin="VCC"/>
+<pinref part="P+6" gate="G$1" pin="+3V3"/>
+<wire x1="93.98" y1="91.44" x2="86.36" y2="91.44" width="0.1524" layer="91"/>
+<wire x1="86.36" y1="91.44" x2="86.36" y2="96.52" width="0.1524" layer="91"/>
+<pinref part="U$1" gate="A" pin="RST"/>
+<wire x1="93.98" y1="86.36" x2="86.36" y2="86.36" width="0.1524" layer="91"/>
+<wire x1="86.36" y1="86.36" x2="86.36" y2="91.44" width="0.1524" layer="91"/>
+<junction x="86.36" y="91.44"/>
+<pinref part="U$1" gate="A" pin="CH_PD"/>
+<wire x1="93.98" y1="81.28" x2="86.36" y2="81.28" width="0.1524" layer="91"/>
+<wire x1="86.36" y1="81.28" x2="86.36" y2="86.36" width="0.1524" layer="91"/>
+<junction x="86.36" y="86.36"/>
+</segment>
+</net>
+<net name="PROGRAM" class="0">
+<segment>
+<pinref part="U$1" gate="A" pin="GPIO0"/>
+<wire x1="129.54" y1="81.28" x2="137.16" y2="81.28" width="0.1524" layer="91"/>
+<label x="137.16" y="81.28" size="1.27" layer="95" xref="yes"/>
+</segment>
+<segment>
+<pinref part="JP2" gate="A" pin="2"/>
+<wire x1="33.02" y1="73.66" x2="22.86" y2="73.66" width="0.1524" layer="91"/>
+<label x="22.86" y="73.66" size="1.27" layer="95" rot="R180" xref="yes"/>
+</segment>
+</net>
+<net name="DATA" class="0">
+<segment>
+<pinref part="U$1" gate="A" pin="DATA/GPIO2"/>
+<wire x1="129.54" y1="76.2" x2="137.16" y2="76.2" width="0.1524" layer="91"/>
+<label x="137.16" y="76.2" size="1.27" layer="95" xref="yes"/>
+</segment>
+<segment>
+<pinref part="JP1" gate="A" pin="2"/>
+<wire x1="121.92" y1="25.4" x2="111.76" y2="25.4" width="0.1524" layer="91"/>
+<label x="111.76" y="25.4" size="1.27" layer="95" rot="R180" xref="yes"/>
+</segment>
+</net>

Commit message: added voltage regulator for 5V and cleaned up schematic
Parts:
- added C3: (no value), rcl:CPOL-EU140CLH-0810
- added C4: 470u, rcl:CPOL-EU140CLH-0810
- added D1: (no value), diode:SCHOTTKY-DIODESMC
- added L1: L-EUPISR, Inductor-Fastron:L-EUPISR
- added U$2: LM2576S5,0, lightstick:LM2576S5,0
Connections:
- new net N$1: D1.C, L1.1, U$2.OUTPUT
- net +12V: now also C3.+, U$2.VIN
- net +5V: now also C4.+, L1.2, U$2.FEEDBACK
- net GND: now also C3.-, C4.-, D1.A, U$2.GND, U$2.GROUND, U$2.OFF
Other:
- note added: "12V -> 5V voltage regulator"
- note added: "TODO: verify device case"
- note added: "power supply 2 connectors to allow daisy chain"
- note removed: "power supply"
- moved on the sheet: C1, C2, U1
