File: hardware/lightstick.sch (EAGLE design)
At the start: 14 parts, among them U1 MCP1703AT-3302E/CB, X1 RIA182-02, X2 RIA182-02

Commit message: added value for C3
Parts:
- C3: value (none) -> 100u
Changed lines of the file:
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@@
 <part name="D1" library="diode" deviceset="SCHOTTKY-DIODE" device="SMC"/>
 <part name="GND13" library="supply1" deviceset="GND" device=""/>
-<part name="C3" library="rcl" deviceset="CPOL-EU" device="140CLH-0810"/>
+<part name="C3" library="rcl" deviceset="CPOL-EU" device="140CLH-0810" value="100u"/>
 <part name="C4" library="rcl" deviceset="CPOL-EU" device="140CLH-0810" value="470u"/>
 <part name="GND14" library="supply1" deviceset="GND" device=""/>

Commit message: changed routing of +5V power line; changed C3, C4 footprint
Parts:
- C3: device rcl:CPOL-EU140CLH-0810 -> rcl:CPOL-EUD
- C4: device rcl:CPOL-EU140CLH-0810 -> rcl:CPOL-EUF
Changed lines of the file:
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@@
 <part name="D1" library="diode" deviceset="SCHOTTKY-DIODE" device="SMC"/>
 <part name="GND13" library="supply1" deviceset="GND" device=""/>
-<part name="C3" library="rcl" deviceset="CPOL-EU" device="140CLH-0810" value="100u"/>
-<part name="C4" library="rcl" deviceset="CPOL-EU" device="140CLH-0810" value="470u"/>
+<part name="C3" library="rcl" deviceset="CPOL-EU" device="D" value="100u"/>
+<part name="C4" library="rcl" deviceset="CPOL-EU" device="F" value="470u"/>
 <part name="GND14" library="supply1" deviceset="GND" device=""/>
 <part name="GND15" library="supply1" deviceset="GND" device=""/>
