File: hardware/lightstick.sch (EAGLE design)
At the start: 14 parts, among them U1 MCP1703AT-3302E/CB, X1 RIA182-02, X2 RIA182-02

Commit message: changed D1 to correct part
Parts:
- D1: device diode:SCHOTTKY-DIODESMC -> diode:DIODE-DO214AC
Other:
- note added: "Schottky Diode"
- note removed: "TODO: verify device case"
Changed lines of the file:
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@@
 <part name="P+7" library="supply1" deviceset="+12V" device=""/>
 <part name="L1" library="Inductor-Fastron" deviceset="L-EU" device="PISR"/>
-<part name="D1" library="diode" deviceset="SCHOTTKY-DIODE" device="SMC"/>
+<part name="D1" library="diode" deviceset="DIODE-" device="DO214AC"/>
 <part name="GND13" library="supply1" deviceset="GND" device=""/>
 <part name="C3" library="rcl" deviceset="CPOL-EU" device="D" value="100u"/>
@@
 <text x="109.22" y="167.64" size="1.27" layer="91">Voltage regulator 5V -&gt; 3V3</text>
 <text x="17.78" y="170.18" size="1.27" layer="91">ESP 8266 controller</text>
-<text x="137.16" y="86.36" size="1.778" layer="91" rot="R90">TODO: verify device case</text>
 <text x="104.14" y="129.54" size="1.778" layer="91">12V -&gt; 5V voltage regulator</text>
+<text x="137.16" y="93.98" size="1.778" layer="91" rot="R90">Schottky Diode</text>
 </plain>
 <instances>

Commit message: changed D1 to MBRS340
Parts:
- D1: value (none) -> MBRS340T3; device diode:DIODE-DO214AC -> diode:MBRS340T3
Other:
- note removed: "Schottky Diode"
Changed lines of the file:
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@@
 <part name="P+7" library="supply1" deviceset="+12V" device=""/>
 <part name="L1" library="Inductor-Fastron" deviceset="L-EU" device="PISR"/>
-<part name="D1" library="diode" deviceset="DIODE-" device="DO214AC"/>
 <part name="GND13" library="supply1" deviceset="GND" device=""/>
 <part name="C3" library="rcl" deviceset="CPOL-EU" device="D" value="100u"/>
@@
 <part name="GND15" library="supply1" deviceset="GND" device=""/>
 <part name="P+8" library="supply1" deviceset="+5V" device=""/>
+<part name="D1" library="diode" deviceset="MBRS3*0T3" device="" technology="4"/>
 </parts>
 <sheets>
@@
 <text x="17.78" y="170.18" size="1.27" layer="91">ESP 8266 controller</text>
 <text x="104.14" y="129.54" size="1.778" layer="91">12V -&gt; 5V voltage regulator</text>
-<text x="137.16" y="93.98" size="1.778" layer="91" rot="R90">Schottky Diode</text>
 </plain>
 <instances>
@@
 <instance part="P+7" gate="1" x="93.98" y="124.46"/>
 <instance part="L1" gate="G$1" x="149.86" y="114.3" rot="R90"/>
-<instance part="D1" gate="G$1" x="139.7" y="106.68" rot="R90"/>
 <instance part="GND13" gate="1" x="139.7" y="91.44"/>
 <instance part="C3" gate="G$1" x="93.98" y="109.22"/>
@@
 <instance part="GND15" gate="1" x="157.48" y="91.44"/>
 <instance part="P+8" gate="1" x="165.1" y="121.92"/>
+<instance part="D1" gate="G$1" x="139.7" y="101.6" rot="R90"/>
 </instances>
 <busses>
@@
 <segment>
 <pinref part="GND13" gate="1" pin="GND"/>
+<wire x1="139.7" y1="93.98" x2="139.7" y2="99.06" width="0.1524" layer="91"/>
 <pinref part="D1" gate="G$1" pin="A"/>
-<wire x1="139.7" y1="93.98" x2="139.7" y2="104.14" width="0.1524" layer="91"/>
 </segment>
 <segment>
@@
 <pinref part="L1" gate="G$1" pin="1"/>
 <wire x1="137.16" y1="114.3" x2="139.7" y2="114.3" width="0.1524" layer="91"/>
+<wire x1="139.7" y1="114.3" x2="144.78" y2="114.3" width="0.1524" layer="91"/>
+<wire x1="139.7" y1="104.14" x2="139.7" y2="114.3" width="0.1524" layer="91"/>
+<junction x="139.7" y="114.3"/>
 <pinref part="D1" gate="G$1" pin="C"/>
-<wire x1="139.7" y1="114.3" x2="144.78" y2="114.3" width="0.1524" layer="91"/>
-<wire x1="139.7" y1="109.22" x2="139.7" y2="114.3" width="0.1524" layer="91"/>
-<junction x="139.7" y="114.3"/>
-</segment>
-</net>
+</segment>
+</net>

Commit message: changed power connector
Parts:
- removed X1, X2: RIA182-02, con-ria182:RIA182-02
- added U$3, U$4: AKL383-02, lightstick:AKL383-02
Connections:
- net +12V: now also U$3.PIN1, U$4.PIN1; no longer X1-1.SK, X2-1.SK
- net +3V3: now also JP2.1
- net +5V: no longer JP2.1
- net GND: now also U$3.PIN2, U$4.PIN2; no longer X1-2.SK, X2-2.SK
Changed lines of the file:
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@@
 <parts>
 <part name="FRAME1" library="frames" deviceset="A4L-LOC" device=""/>
-<part name="X1" library="con-ria182" deviceset="RIA182-02" device=""/>
-<part name="X2" library="con-ria182" deviceset="RIA182-02" device=""/>
 <part name="P+1" library="supply1" deviceset="+12V" device=""/>
 <part name="P+2" library="supply1" deviceset="+12V" device=""/>
@@
 <part name="P+8" library="supply1" deviceset="+5V" device=""/>
 <part name="D1" library="diode" deviceset="MBRS3*0T3" device="" technology="4"/>
+<part name="U$3" library="lightstick" deviceset="AKL383-02" device=""/>
+<part name="U$4" library="lightstick" deviceset="AKL383-02" device=""/>
 </parts>
 <sheets>
@@
 <instances>
 <instance part="FRAME1" gate="G$1" x="0" y="0"/>
-<instance part="X1" gate="-1" x="22.86" y="27.94"/>
-<instance part="X1" gate="-2" x="22.86" y="22.86"/>
-<instance part="X2" gate="-1" x="48.26" y="27.94"/>
-<instance part="X2" gate="-2" x="48.26" y="22.86"/>
 <instance part="P+1" gate="1" x="30.48" y="35.56"/>
 <instance part="P+2" gate="1" x="55.88" y="35.56"/>
@@
 <instance part="P+8" gate="1" x="165.1" y="121.92"/>
 <instance part="D1" gate="G$1" x="139.7" y="101.6" rot="R90"/>
+<instance part="U$3" gate="G$1" x="40.64" y="22.86"/>
+<instance part="U$4" gate="G$1" x="12.7" y="22.86"/>
 </instances>
 <busses>
@@
 <net name="GND" class="0">
 <segment>
-<pinref part="X1" gate="-2" pin="SK"/>
-<pinref part="GND1" gate="1" pin="GND"/>
-<wire x1="27.94" y1="22.86" x2="30.48" y2="22.86" width="0.1524" layer="91"/>
-<wire x1="30.48" y1="22.86" x2="30.48" y2="17.78" width="0.1524" layer="91"/>
-</segment>
-<segment>
-<pinref part="X2" gate="-2" pin="SK"/>
 <pinref part="GND2" gate="1" pin="GND"/>
 <wire x1="53.34" y1="22.86" x2="55.88" y2="22.86" width="0.1524" layer="91"/>
 <wire x1="55.88" y1="22.86" x2="55.88" y2="17.78" width="0.1524" layer="91"/>
+<pinref part="U$3" gate="G$1" pin="PIN2"/>
 </segment>
 <segment>
@@
 <wire x1="157.48" y1="101.6" x2="157.48" y2="93.98" width="0.1524" layer="91"/>
 </segment>
+<segment>
+<pinref part="U$4" gate="G$1" pin="PIN2"/>
+<pinref part="GND1" gate="1" pin="GND"/>
+<wire x1="30.48" y1="17.78" x2="30.48" y2="22.86" width="0.1524" layer="91"/>
+<wire x1="30.48" y1="22.86" x2="25.4" y2="22.86" width="0.1524" layer="91"/>
+</segment>
 </net>
 <net name="+12V" class="0">
 <segment>
-<pinref part="X1" gate="-1" pin="SK"/>
-<pinref part="P+1" gate="1" pin="+12V"/>
-<wire x1="27.94" y1="27.94" x2="30.48" y2="27.94" width="0.1524" layer="91"/>
-<wire x1="30.48" y1="27.94" x2="30.48" y2="33.02" width="0.1524" layer="91"/>
-</segment>
-<segment>
-<pinref part="X2" gate="-1" pin="SK"/>
 <pinref part="P+2" gate="1" pin="+12V"/>
 <wire x1="53.34" y1="27.94" x2="55.88" y2="27.94" width="0.1524" layer="91"/>
 <wire x1="55.88" y1="27.94" x2="55.88" y2="33.02" width="0.1524" layer="91"/>
+<pinref part="U$3" gate="G$1" pin="PIN1"/>
 </segment>
 <segment>
@@
 <junction x="93.98" y="116.84"/>
 </segment>
+<segment>
+<pinref part="U$4" gate="G$1" pin="PIN1"/>
+<pinref part="P+1" gate="1" pin="+12V"/>
+<wire x1="30.48" y1="33.02" x2="30.48" y2="27.94" width="0.1524" layer="91"/>
+<wire x1="30.48" y1="27.94" x2="25.4" y2="27.94" width="0.1524" layer="91"/>
+</segment>
 </net>
 <net name="+5V" class="0">
@@
 <wire x1="121.92" y1="27.94" x2="111.76" y2="27.94" width="0.1524" layer="91"/>
 <wire x1="111.76" y1="27.94" x2="111.76" y2="30.48" width="0.1524" layer="91"/>
-</segment>
-<segment>
-<pinref part="JP2" gate="A" pin="1"/>
-<pinref part="P+4" gate="G$1" pin="+3V3"/>
-<wire x1="33.02" y1="76.2" x2="22.86" y2="76.2" width="0.1524" layer="91"/>
-<wire x1="22.86" y1="76.2" x2="22.86" y2="78.74" width="0.1524" layer="91"/>
 </segment>
 <segment>
@@
 <junction x="10.16" y="157.48"/>
 </segment>
-</net>
+<segment>
+<pinref part="P+4" gate="G$1" pin="+3V3"/>
+<pinref part="JP2" gate="A" pin="1"/>
+<wire x1="22.86" y1="78.74" x2="22.86" y2="76.2" width="0.1524" layer="91"/>
+<wire x1="22.86" y1="76.2" x2="33.02" y2="76.2" width="0.1524" layer="91"/>
+</segment>
+</net>

Commit message: rerouting to accomodate easier soldering. connected GND top and bottom planes
Parts:
- added JP4: (no value), pinhead:PINHD-1X1
Connections:
- net GND: now also JP4.1
Other:
- note added: "connection GND top side / bottom side"
Changed lines of the file:
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@@
 <part name="U$3" library="lightstick" deviceset="AKL383-02" device=""/>
 <part name="U$4" library="lightstick" deviceset="AKL383-02" device=""/>
+<part name="JP4" library="pinhead" deviceset="PINHD-1X1" device=""/>
+<part name="GND16" library="supply1" deviceset="GND" device=""/>
 </parts>
 <sheets>
@@
 <text x="17.78" y="170.18" size="1.27" layer="91">ESP 8266 controller</text>
 <text x="104.14" y="129.54" size="1.778" layer="91">12V -&gt; 5V voltage regulator</text>
+<text x="91.44" y="76.2" size="1.778" layer="91">connection GND top side / bottom side</text>
 </plain>
 <instances>
@@
 <instance part="U$3" gate="G$1" x="40.64" y="22.86"/>
 <instance part="U$4" gate="G$1" x="12.7" y="22.86"/>
+<instance part="JP4" gate="G$1" x="124.46" y="63.5"/>
+<instance part="GND16" gate="1" x="111.76" y="55.88"/>
 </instances>
 <busses>
@@
 <wire x1="30.48" y1="17.78" x2="30.48" y2="22.86" width="0.1524" layer="91"/>
 <wire x1="30.48" y1="22.86" x2="25.4" y2="22.86" width="0.1524" layer="91"/>
+</segment>
+<segment>
+<pinref part="JP4" gate="G$1" pin="1"/>
+<pinref part="GND16" gate="1" pin="GND"/>
+<wire x1="121.92" y1="63.5" x2="111.76" y2="63.5" width="0.1524" layer="91" style="longdash"/>
+<wire x1="111.76" y1="63.5" x2="111.76" y2="58.42" width="0.1524" layer="91" style="longdash"/>
 </segment>
 </net>
@@
 <wire x1="137.16" y1="45.72" x2="137.16" y2="5.08" width="0.1524" layer="91" style="longdash"/>
 <wire x1="86.36" y1="45.72" x2="86.36" y2="5.08" width="0.1524" layer="91" style="longdash"/>
-<wire x1="86.36" y1="45.72" x2="86.36" y2="172.72" width="0.1524" layer="91" style="longdash"/>
-<wire x1="170.18" y1="45.72" x2="170.18" y2="172.72" width="0.1524" layer="91" style="longdash"/>
+<wire x1="86.36" y1="45.72" x2="86.36" y2="81.28" width="0.1524" layer="91" style="longdash"/>
+<wire x1="86.36" y1="81.28" x2="86.36" y2="172.72" width="0.1524" layer="91" style="longdash"/>
+<wire x1="170.18" y1="45.72" x2="170.18" y2="81.28" width="0.1524" layer="91" style="longdash"/>
+<wire x1="170.18" y1="81.28" x2="170.18" y2="172.72" width="0.1524" layer="91" style="longdash"/>
 <wire x1="137.16" y1="45.72" x2="170.18" y2="45.72" width="0.1524" layer="91" style="longdash"/>
+<wire x1="86.36" y1="81.28" x2="170.18" y2="81.28" width="0.1524" layer="91" style="longdash"/>
 </segment>
 </net>
@@
 </sheet>
 </sheets>
+<errors>
+</errors>
 </schematic>
 </drawing>
