File: hardware/lightstick.brd (EAGLE design)
At the start: 55 x 35 mm, 14 parts, among them U1 MCP1703AT-3302E/CB, X1 RIA182-02, X2 RIA182-02

Commit message: new layout + routing
Parts:
- moved X2 44.9 mm to (7.04, 23.2), turned to 270 degrees
- moved JP3 32.6 mm to (39.7, 4.73)
- moved C4 26.2 mm to (27.4, 29.6)
- moved JP2 25.8 mm to (39.7, 24.4)
- moved C1 19.5 mm to (22.6, 15.8), flipped to the bottom
- moved C2 18.3 mm to (32.8, 15.0), flipped to the bottom, turned to 270 degrees
- moved U1 17.5 mm to (28.5, 14.7), flipped to the bottom
- moved D1 16.4 mm to (14.2, 12.1), turned to 270 degrees
- moved JP1 13.6 mm to (37.3, 31.6), turned to 0 degrees
- moved U$1 13.5 mm to (30.3, 14.5)
- moved U$2 12.5 mm to (15.9, 28.5), turned to 270 degrees
- moved C3 11.8 mm to (14.8, 28.9), flipped to the bottom
- moved L1 11.4 mm to (28.6, 14.2)
- moved X1 0.72 mm to (7.02, 13.9)
Routing:
- net +5V: track 0.00 -> 50.9 mm, vias 0 -> 1
- net DATA: track 0.00 -> 44.4 mm
- net +3V3: track 0.00 -> 34.3 mm
- net +12V: track 0.00 -> 24.0 mm
- net N$1: track 0.00 -> 22.7 mm
- net TX: track 0.00 -> 16.0 mm
- net PROGRAM: track 0.00 -> 13.9 mm
- net RX: track 0.00 -> 6.25 mm
Other:
- board size 55 x 35 mm -> 50 x 35 mm
- board text added: "C3MA Lightstick 20150412"

Commit message: added value for C3
Parts:
- C3: value (none) -> 100u
Routing:
- net +12V: track 24.0 -> 23.1 mm
Changed lines of the file:
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@@
 <element name="L1" library="Inductor-Fastron" package="PISR" value="L-EUPISR" x="28.61" y="14.23" rot="R90"/>
 <element name="D1" library="diode" package="SMC" value="" x="14.22" y="12.07" rot="R270"/>
-<element name="C3" library="rcl" package="140CLH-0810" value="" x="14.76" y="28.92" rot="MR270"/>
+<element name="C3" library="rcl" package="140CLH-0810" value="100u" x="14.76" y="28.92" rot="MR270"/>
 <element name="C4" library="rcl" package="140CLH-0810" value="470u" x="27.35" y="29.58"/>
 </elements>
@@
 <contactref element="U$2" pad="VIN"/>
 <contactref element="C3" pad="+"/>
-<wire x1="7.04" y1="23.17" x2="9.5579" y2="23.17" width="1.016" layer="1"/>
-<wire x1="9.5579" y1="23.17" x2="12.5264" y2="20.2015" width="1.016" layer="1"/>
 <wire x1="14.76" y1="25.67" x2="9.54" y2="25.67" width="1.016" layer="16"/>
 <wire x1="9.54" y1="25.67" x2="7.04" y2="23.17" width="1.016" layer="16"/>
-<wire x1="7.02" y1="13.94" x2="12.5264" y2="19.4464" width="1.016" layer="1"/>
 <wire x1="12.5264" y1="19.4464" x2="12.5264" y2="20.2015" width="0.4064" layer="1"/>
+<wire x1="7.02" y1="13.94" x2="10.8" y2="17.72" width="1.6764" layer="1"/>
+<wire x1="10.8" y1="17.72" x2="10.8" y2="21.5" width="1.6764" layer="1"/>
+<wire x1="10.8" y1="21.5" x2="9.13" y2="23.17" width="1.6764" layer="1"/>
+<wire x1="9.13" y1="23.17" x2="7.04" y2="23.17" width="1.6764" layer="1"/>
+<wire x1="10.8" y1="21.5" x2="12.5264" y2="20.2015" width="0" layer="19" extent="1-1"/>
 </signal>
 <signal name="+5V">

Commit message: changed routing of +5V power line; changed C3, C4 footprint
Parts:
- C3: device rcl:140CLH-0810 -> rcl:PANASONIC_D
- C4: device rcl:140CLH-0810 -> rcl:PANASONIC_F
- moved C1 3.06 mm to (23.8, 13.0), turned to 270 degrees
Routing:
- net +5V: track 50.9 -> 55.8 mm
- net +12V: track 23.1 -> 26.7 mm
Changed lines of the file:
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@@
 <attribute name="OC_FARNELL" value="2218573" x="67.91" y="60.41" size="1.778" layer="28" rot="MR180" display="off"/>
 </element>
-<element name="C1" library="rcl" package="C0805" value="1u" x="22.61" y="15.85" rot="MR0"/>
+<element name="C1" library="rcl" package="C0805" value="1u" x="23.75" y="13.01" rot="MR270"/>
 <element name="C2" library="rcl" package="C0805" value="1u" x="32.76" y="15.01" rot="MR270"/>
 <element name="U$1" library="lightstick" package="ESP8266" value="ESP8266" x="30.34" y="14.47" rot="MR270"/>
@@
 <element name="L1" library="Inductor-Fastron" package="PISR" value="L-EUPISR" x="28.61" y="14.23" rot="R90"/>
 <element name="D1" library="diode" package="SMC" value="" x="14.22" y="12.07" rot="R270"/>
-<element name="C3" library="rcl" package="140CLH-0810" value="100u" x="14.76" y="28.92" rot="MR270"/>
-<element name="C4" library="rcl" package="140CLH-0810" value="470u" x="27.35" y="29.58"/>
+<element name="C3" library="rcl" package="PANASONIC_D" value="100u" x="14.76" y="28.92" rot="MR270"/>
+<element name="C4" library="rcl" package="PANASONIC_F" value="470u" x="27.35" y="29.58"/>
 </elements>
 <signals>
@@
 <contactref element="U$2" pad="VIN"/>
 <contactref element="C3" pad="+"/>
-<wire x1="14.76" y1="25.67" x2="9.54" y2="25.67" width="1.016" layer="16"/>
-<wire x1="9.54" y1="25.67" x2="7.04" y2="23.17" width="1.016" layer="16"/>
 <wire x1="12.5264" y1="19.4464" x2="12.5264" y2="20.2015" width="0.4064" layer="1"/>
 <wire x1="7.02" y1="13.94" x2="10.8" y2="17.72" width="1.6764" layer="1"/>
 <wire x1="10.8" y1="17.72" x2="10.8" y2="21.5" width="1.6764" layer="1"/>
-<wire x1="10.8" y1="21.5" x2="9.13" y2="23.17" width="1.6764" layer="1"/>
+<wire x1="10.8" y1="21.5" x2="10.35" y2="21.95" width="1.6764" layer="1"/>
+<wire x1="10.35" y1="21.95" x2="9.13" y2="23.17" width="1.6764" layer="1"/>
 <wire x1="9.13" y1="23.17" x2="7.04" y2="23.17" width="1.6764" layer="1"/>
-<wire x1="10.8" y1="21.5" x2="12.5264" y2="20.2015" width="0" layer="19" extent="1-1"/>
+<wire x1="7.04" y1="23.17" x2="7.17" y2="23.17" width="0.4064" layer="1"/>
+<wire x1="7.17" y1="23.17" x2="7.3" y2="23.3" width="0.4064" layer="1"/>
+<wire x1="14.76" y1="26.52" x2="10.39" y2="26.52" width="0.6096" layer="16"/>
+<wire x1="10.39" y1="26.52" x2="7.04" y2="23.17" width="0.6096" layer="16"/>
+<wire x1="12.5264" y1="20.2015" x2="12.0985" y2="20.2015" width="1.27" layer="1"/>
+<wire x1="12.0985" y1="20.2015" x2="10.35" y2="21.95" width="1.27" layer="1"/>
 </signal>
 <signal name="+5V">
@@
 <contactref element="U$2" pad="FEEDBACK"/>
 <contactref element="C4" pad="+"/>
-<wire x1="23.56" y1="15.85" x2="25.9138" y2="13.4962" width="0.4064" layer="16"/>
-<wire x1="25.9138" y1="13.4962" x2="28.54" y2="13.4962" width="0.4064" layer="16"/>
 <wire x1="17.6318" y1="20.2015" x2="17.6318" y2="18.5682" width="0.4064" layer="1"/>
-<wire x1="17.6318" y1="18.5682" x2="18.6" y2="17.6" width="0.4064" layer="1"/>
-<via x="18.6" y="17.6" extent="1-16" drill="0.7"/>
-<wire x1="17.6318" y1="20.2015" x2="17.6318" y2="21.6318" width="1.6764" layer="1"/>
-<wire x1="17.6318" y1="21.6318" x2="18.4" y2="22.4" width="1.6764" layer="1"/>
-<wire x1="18.4" y1="22.4" x2="28.24" y2="22.4" width="1.6764" layer="1"/>
+<via x="19.5" y="14.5" extent="1-16" drill="0.7"/>
 <wire x1="28.24" y1="22.4" x2="28.61" y2="22.03" width="0.6096" layer="1"/>
 <wire x1="28.24" y1="22.4" x2="28.24" y2="27.22" width="1.6764" layer="1"/>
-<wire x1="28.24" y1="27.22" x2="30.6" y2="29.58" width="1.6764" layer="1"/>
-<wire x1="34.8" y1="31.63" x2="32.65" y2="31.63" width="1.6764" layer="1"/>
-<wire x1="32.65" y1="31.63" x2="30.6" y2="29.58" width="1.6764" layer="1"/>
 <wire x1="37.18" y1="24.43" x2="31.01" y2="24.43" width="0.6096" layer="1"/>
 <wire x1="31.01" y1="24.43" x2="28.61" y2="22.03" width="0.6096" layer="1"/>
-<wire x1="18.6" y1="17.6" x2="22.9" y2="17.6" width="0.4064" layer="16"/>
-<wire x1="22.9" y1="17.6" x2="23.56" y2="16.94" width="0.4064" layer="16"/>
-<wire x1="23.56" y1="16.94" x2="23.56" y2="15.85" width="0.4064" layer="16"/>
+<wire x1="34.8" y1="31.63" x2="32.95" y2="31.63" width="1.6764" layer="1"/>
+<wire x1="32.95" y1="31.63" x2="30.9" y2="29.58" width="1.6764" layer="1"/>
+<wire x1="28.24" y1="27.22" x2="28.54" y2="27.22" width="1.6764" layer="1"/>
+<wire x1="28.54" y1="27.22" x2="30.9" y2="29.58" width="1.6764" layer="1"/>
+<wire x1="17.6318" y1="20.2015" x2="17.6318" y2="17.9682" width="1.6764" layer="1"/>
+<wire x1="17.6318" y1="17.9682" x2="18.1" y2="17.5" width="1.6764" layer="1"/>
+<wire x1="18.1" y1="17.5" x2="18.5" y2="17.1" width="1.6764" layer="1"/>
+<wire x1="18.5" y1="17.1" x2="27.4" y2="17.1" width="1.6764" layer="1"/>
+<wire x1="27.4" y1="17.1" x2="28.6" y2="18.3" width="1.6764" layer="1"/>
+<wire x1="28.6" y1="18.3" x2="28.6" y2="22.02" width="1.6764" layer="1"/>
+<wire x1="28.6" y1="22.02" x2="28.61" y2="22.03" width="1.6764" layer="1"/>
+<wire x1="28.54" y1="13.4962" x2="28.0762" y2="13.96" width="0.4064" layer="16"/>
+<wire x1="28.0762" y1="13.96" x2="23.75" y2="13.96" width="0.4064" layer="16"/>
+<wire x1="23.75" y1="13.96" x2="20.04" y2="13.96" width="0.4064" layer="16"/>
+<wire x1="20.04" y1="13.96" x2="19.5" y2="14.5" width="0.4064" layer="16"/>
+<wire x1="19.5" y1="14.5" x2="18.1" y2="15.9" width="0.4064" layer="1"/>
+<wire x1="18.1" y1="15.9" x2="18.1" y2="17.5" width="0.4064" layer="1"/>
 </signal>
 <signal name="RX">

Commit message: changed D1 to correct part
Parts:
- D1: device diode:SMC -> diode:DO214AC
Routing:
- net N$1: track 22.7 -> 23.7 mm
Changed lines of the file:
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@@
 <element name="U$2" library="lightstick" package="TO-263" value="LM2576S5,0" x="15.93" y="28.52" rot="R270"/>
 <element name="L1" library="Inductor-Fastron" package="PISR" value="L-EUPISR" x="28.61" y="14.23" rot="R90"/>
-<element name="D1" library="diode" package="SMC" value="" x="14.22" y="12.07" rot="R270"/>
+<element name="D1" library="diode" package="DO214AC" value="" x="14.22" y="12.07" rot="R270"/>
 <element name="C3" library="rcl" package="PANASONIC_D" value="100u" x="14.76" y="28.92" rot="MR270"/>
 <element name="C4" library="rcl" package="PANASONIC_F" value="470u" x="27.35" y="29.58"/>
@@
 <contactref element="D1" pad="C"/>
 <wire x1="14.2282" y1="20.2015" x2="14.22" y2="20.1933" width="0.4064" layer="1"/>
-<wire x1="14.22" y1="20.1933" x2="14.22" y2="15.77" width="1.6764" layer="1"/>
-<wire x1="14.22" y1="15.77" x2="23.56" y2="6.43" width="1.6764" layer="1"/>
-<wire x1="23.56" y1="6.43" x2="28.61" y2="6.43" width="1.6764" layer="1"/>
+<wire x1="21.91" y1="6.43" x2="28.61" y2="6.43" width="1.6764" layer="1"/>
+<wire x1="14.22" y1="14.12" x2="14.22" y2="20.2015" width="1.6764" layer="1"/>
+<wire x1="14.22" y1="20.2015" x2="14.2282" y2="20.2015" width="1.6764" layer="1"/>
+<wire x1="21.91" y1="6.43" x2="14.22" y2="14.12" width="1.6764" layer="1"/>
 </signal>
 </signals>

Commit message: changed D1 to MBRS340
Parts:
- D1: value (none) -> MBRS340T3; device diode:DO214AC -> diode:SMC
- moved D1 0.93 mm to (13.9, 11.2)
Routing:
- net +5V: track 55.8 -> 51.7 mm
Changed lines of the file:
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@@
 <element name="U$2" library="lightstick" package="TO-263" value="LM2576S5,0" x="15.93" y="28.52" rot="R270"/>
 <element name="L1" library="Inductor-Fastron" package="PISR" value="L-EUPISR" x="28.61" y="14.23" rot="R90"/>
-<element name="D1" library="diode" package="DO214AC" value="" x="14.22" y="12.07" rot="R270"/>
 <element name="C3" library="rcl" package="PANASONIC_D" value="100u" x="14.76" y="28.92" rot="MR270"/>
 <element name="C4" library="rcl" package="PANASONIC_F" value="470u" x="27.35" y="29.58"/>
+<element name="D1" library="diode" package="SMC" value="MBRS340T3" x="13.9" y="11.2" rot="R270"/>
 </elements>
 <signals>
@@
 <contactref element="U$2" pad="GND"/>
 <contactref element="U$2" pad="OFF"/>
-<contactref element="D1" pad="A"/>
 <contactref element="C3" pad="-"/>
 <contactref element="C4" pad="-"/>
@@
 <vertex x="0" y="35"/>
 </polygon>
+<contactref element="D1" pad="A"/>
 </signal>
 <signal name="+12V">
@@
 <contactref element="U$2" pad="FEEDBACK"/>
 <contactref element="C4" pad="+"/>
-<wire x1="17.6318" y1="20.2015" x2="17.6318" y2="18.5682" width="0.4064" layer="1"/>
 <via x="19.5" y="14.5" extent="1-16" drill="0.7"/>
-<wire x1="28.24" y1="22.4" x2="28.61" y2="22.03" width="0.6096" layer="1"/>
 <wire x1="28.24" y1="22.4" x2="28.24" y2="27.22" width="1.6764" layer="1"/>
 <wire x1="37.18" y1="24.43" x2="31.01" y2="24.43" width="0.6096" layer="1"/>
@@
 <wire x1="28.24" y1="27.22" x2="28.54" y2="27.22" width="1.6764" layer="1"/>
 <wire x1="28.54" y1="27.22" x2="30.9" y2="29.58" width="1.6764" layer="1"/>
-<wire x1="17.6318" y1="20.2015" x2="17.6318" y2="17.9682" width="1.6764" layer="1"/>
-<wire x1="17.6318" y1="17.9682" x2="18.1" y2="17.5" width="1.6764" layer="1"/>
-<wire x1="18.1" y1="17.5" x2="18.5" y2="17.1" width="1.6764" layer="1"/>
-<wire x1="18.5" y1="17.1" x2="27.4" y2="17.1" width="1.6764" layer="1"/>
-<wire x1="27.4" y1="17.1" x2="28.6" y2="18.3" width="1.6764" layer="1"/>
-<wire x1="28.6" y1="18.3" x2="28.6" y2="22.02" width="1.6764" layer="1"/>
 <wire x1="28.6" y1="22.02" x2="28.61" y2="22.03" width="1.6764" layer="1"/>
 <wire x1="28.54" y1="13.4962" x2="28.0762" y2="13.96" width="0.4064" layer="16"/>
@@
 <wire x1="23.75" y1="13.96" x2="20.04" y2="13.96" width="0.4064" layer="16"/>
 <wire x1="20.04" y1="13.96" x2="19.5" y2="14.5" width="0.4064" layer="16"/>
-<wire x1="19.5" y1="14.5" x2="18.1" y2="15.9" width="0.4064" layer="1"/>
-<wire x1="18.1" y1="15.9" x2="18.1" y2="17.5" width="0.4064" layer="1"/>
+<wire x1="17.6318" y1="20.2015" x2="17.6318" y2="21.7318" width="0.6096" layer="1"/>
+<wire x1="17.6318" y1="21.7318" x2="18.3" y2="22.4" width="0.6096" layer="1"/>
+<wire x1="18.3" y1="22.4" x2="28.24" y2="22.4" width="0.6096" layer="1"/>
+<wire x1="28.24" y1="22.4" x2="28.61" y2="22.03" width="0.6096" layer="1"/>
+<wire x1="19.5" y1="14.5" x2="17.6318" y2="16.3682" width="0.6096" layer="1"/>
+<wire x1="17.6318" y1="16.3682" x2="17.6318" y2="20.2015" width="0.6096" layer="1"/>
 </signal>
 <signal name="RX">
@@
 <contactref element="U$2" pad="OUTPUT"/>
 <contactref element="L1" pad="1"/>
-<contactref element="D1" pad="C"/>
 <wire x1="14.2282" y1="20.2015" x2="14.22" y2="20.1933" width="0.4064" layer="1"/>
 <wire x1="21.91" y1="6.43" x2="28.61" y2="6.43" width="1.6764" layer="1"/>
-<wire x1="14.22" y1="14.12" x2="14.22" y2="20.2015" width="1.6764" layer="1"/>
-<wire x1="14.22" y1="20.2015" x2="14.2282" y2="20.2015" width="1.6764" layer="1"/>
-<wire x1="21.91" y1="6.43" x2="14.22" y2="14.12" width="1.6764" layer="1"/>
+<contactref element="D1" pad="C"/>
+<wire x1="21.91" y1="6.43" x2="13.9" y2="14.44" width="1.6764" layer="1"/>
+<wire x1="13.9" y1="14.44" x2="13.9" y2="14.9" width="1.6764" layer="1"/>
+<wire x1="14.2282" y1="20.2015" x2="14.2282" y2="14.9" width="1.6764" layer="1"/>
+<wire x1="14.2282" y1="14.9" x2="13.9" y2="14.9" width="1.6764" layer="1"/>
 </signal>
 </signals>

Commit message: changed power connector
Parts:
- removed X1, X2: RIA182-02, con-ria182:RIA182-02
- added U$3, U$4: AKL383-02, lightstick:AKL383-02
Connections:
- net +12V: now also U$3.PAD1, U$4.PAD1; no longer X1.1, X2.1
- net +3V3: now also JP2.1
- net +5V: no longer JP2.1
- net GND: now also U$3.PAD2, U$4.PAD2; no longer X1.2, X2.2
Routing:
- net +5V: track 51.7 -> 42.1 mm
- net +12V: track 26.7 -> 35.3 mm
- net +3V3: track 34.3 -> 37.8 mm
Changed lines of the file:
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@@
 <hole x="46" y="30.5" drill="3.2"/>
 <hole x="46" y="4.5" drill="3.2"/>
-<text x="9.3" y="2.1" size="1.27" layer="1" font="vector" ratio="12">C3MA Lightstick 20150412</text>
+<text x="9.3" y="2.1" size="1.27" layer="1" font="vector" ratio="15">C3MA Lightstick 20150412</text>
 </plain>
 <attributes>
@@
 </autorouter>
 <elements>
-<element name="X1" library="con-ria182" package="RIA182-02" value="RIA182-02" x="7.02" y="13.94" rot="R270"/>
-<element name="X2" library="con-ria182" package="RIA182-02" value="RIA182-02" x="7.04" y="23.17" rot="R270"/>
 <element name="JP1" library="pinhead" package="1X03" value="" x="37.34" y="31.63"/>
 <element name="JP2" library="pinhead" package="1X03" value="" x="39.72" y="24.43"/>
@@
 <element name="C4" library="rcl" package="PANASONIC_F" value="470u" x="27.35" y="29.58"/>
 <element name="D1" library="diode" package="SMC" value="MBRS340T3" x="13.9" y="11.2" rot="R270"/>
+<element name="U$3" library="lightstick" package="AKL383-02" value="AKL383-02" x="3.9" y="22.7" rot="R270"/>
+<element name="U$4" library="lightstick" package="AKL383-02" value="AKL383-02" x="3.9" y="13" rot="R270"/>
 </elements>
 <signals>
 <signal name="GND">
-<contactref element="X1" pad="2"/>
-<contactref element="X2" pad="2"/>
 <contactref element="JP1" pad="3"/>
 <contactref element="JP2" pad="3"/>
@@
 </polygon>
 <contactref element="D1" pad="A"/>
+<contactref element="U$3" pad="PAD2"/>
+<contactref element="U$4" pad="PAD2"/>
 </signal>
 <signal name="+12V">
-<contactref element="X1" pad="1"/>
-<contactref element="X2" pad="1"/>
 <contactref element="U$2" pad="VIN"/>
 <contactref element="C3" pad="+"/>
 <wire x1="12.5264" y1="19.4464" x2="12.5264" y2="20.2015" width="0.4064" layer="1"/>
-<wire x1="7.02" y1="13.94" x2="10.8" y2="17.72" width="1.6764" layer="1"/>
 <wire x1="10.8" y1="17.72" x2="10.8" y2="21.5" width="1.6764" layer="1"/>
 <wire x1="10.8" y1="21.5" x2="10.35" y2="21.95" width="1.6764" layer="1"/>
-<wire x1="10.35" y1="21.95" x2="9.13" y2="23.17" width="1.6764" layer="1"/>
-<wire x1="9.13" y1="23.17" x2="7.04" y2="23.17" width="1.6764" layer="1"/>
-<wire x1="7.04" y1="23.17" x2="7.17" y2="23.17" width="0.4064" layer="1"/>
-<wire x1="7.17" y1="23.17" x2="7.3" y2="23.3" width="0.4064" layer="1"/>
 <wire x1="14.76" y1="26.52" x2="10.39" y2="26.52" width="0.6096" layer="16"/>
-<wire x1="10.39" y1="26.52" x2="7.04" y2="23.17" width="0.6096" layer="16"/>
 <wire x1="12.5264" y1="20.2015" x2="12.0985" y2="20.2015" width="1.27" layer="1"/>
 <wire x1="12.0985" y1="20.2015" x2="10.35" y2="21.95" width="1.27" layer="1"/>
+<contactref element="U$3" pad="PAD1"/>
+<contactref element="U$4" pad="PAD1"/>
+<wire x1="3.9" y1="24.605" x2="7.695" y2="24.605" width="1.6764" layer="1"/>
+<wire x1="7.695" y1="24.605" x2="10.35" y2="21.95" width="1.6764" layer="1"/>
+<wire x1="3.9" y1="14.905" x2="7.985" y2="14.905" width="1.6764" layer="1"/>
+<wire x1="7.985" y1="14.905" x2="10.8" y2="17.72" width="1.6764" layer="1"/>
+<wire x1="10.39" y1="26.52" x2="8.475" y2="24.605" width="0.6096" layer="16"/>
+<wire x1="8.475" y1="24.605" x2="3.9" y2="24.605" width="0.6096" layer="16"/>
 </signal>
 <signal name="+5V">
 <contactref element="JP1" pad="1"/>
-<contactref element="JP2" pad="1"/>
 <contactref element="C1" pad="1"/>
 <contactref element="U1" pad="3"/>
@@
 <via x="19.5" y="14.5" extent="1-16" drill="0.7"/>
 <wire x1="28.24" y1="22.4" x2="28.24" y2="27.22" width="1.6764" layer="1"/>
-<wire x1="37.18" y1="24.43" x2="31.01" y2="24.43" width="0.6096" layer="1"/>
-<wire x1="31.01" y1="24.43" x2="28.61" y2="22.03" width="0.6096" layer="1"/>
 <wire x1="34.8" y1="31.63" x2="32.95" y2="31.63" width="1.6764" layer="1"/>
 <wire x1="32.95" y1="31.63" x2="30.9" y2="29.58" width="1.6764" layer="1"/>
@@
 <wire x1="43.4" y1="20.1" x2="43.4" y2="13.56" width="0.4064" layer="16"/>
 <wire x1="43.4" y1="13.56" x2="40.5" y2="10.66" width="0.4064" layer="16"/>
+<contactref element="JP2" pad="1"/>
+<wire x1="37.18" y1="24.43" x2="37.18" y2="23.18" width="0.4064" layer="16"/>
+<wire x1="37.18" y1="23.18" x2="35.6" y2="21.6" width="0.4064" layer="16"/>
 </signal>
 <signal name="PROGRAM">
