File: hardware/lightstick.brd (EAGLE design)
At the start: 50 x 35 mm, 14 parts, among them U1 MCP1703AT-3302E/CB

Commit message: rerouting to accomodate easier soldering. connected GND top and bottom planes
Parts:
- added JP4: (no value), pinhead:1X01
- moved C2 6.76 mm to (28.6, 20.3)
- moved JP2 1.71 mm to (38.0, 24.6), turned to 180 degrees
- flipped JP1 to the bottom, turned to 180 degrees
- flipped JP3 to the bottom, turned to 180 degrees
Connections:
- net GND: now also JP4.1
Routing:
- net +3V3: track 37.8 -> 56.7 mm, vias 0 -> 2
- net DATA: track 44.4 -> 29.1 mm
- net PROGRAM: track 13.9 -> 19.5 mm
- net TX: track 16.0 -> 21.3 mm
- net +12V: track 35.3 -> 32.2 mm, vias 0 -> 1
