File: powersupply/lightstick.brd (EAGLE design)
At the start: 50 x 35 mm, 15 parts, among them U1 MCP1703AT-3302E/CB

Commit message: Board modified for new inductor, changed side of capacitor
Parts:
- L1: value L-EUPISR -> L-PWRIND12X12X7; device Inductor-Fastron:PISR -> l-pwr-ind-lib:L12X12X7
- moved C3 24.1 mm to (7.74, 5.88), flipped to the top, turned to 90 degrees
- moved L1 7.46 mm to (26.4, 7.10), turned to 270 degrees
- moved U$3 2.82 mm to (3.10, 25.4)
- moved U$4 2.28 mm to (3.00, 15.1)
Connections:
- net +5V: now also L1.P$2; no longer L1.2
- net N$1: now also L1.P$1; no longer L1.1
Routing:
- net +5V: track 41.7 -> 54.5 mm
- net N$1: track 24.1 -> 16.2 mm
- net +12V: track 32.2 -> 31.2 mm, vias 1 -> 0
Other:
- board text added: "C3MA Lightstick 20150714"
- board text removed: "C3MA Lightstick 20150703"
Changed lines of the file:
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@@
 <?xml version="1.0" encoding="utf-8"?>
 <!DOCTYPE eagle SYSTEM "eagle.dtd">
-<eagle version="6.6.0">
+<eagle version="6.4">
 <drawing>
 <settings>
@@
 <wire x1="50" y1="35" x2="0" y2="35" width="0" layer="20"/>
 <wire x1="0" y1="35" x2="0" y2="0" width="0" layer="20"/>
-<hole x="6" y="4.5" drill="3.2"/>
-<hole x="6" y="30.5" drill="3.2"/>
-<hole x="46" y="30.5" drill="3.2"/>
-<hole x="46" y="4.5" drill="3.2"/>
-<text x="9.3" y="2.1" size="1.27" layer="1" font="vector" ratio="15">C3MA Lightstick 20150703</text>
+<hole x="2.4" y="2" drill="3.2"/>
+<hole x="2.3" y="33.1" drill="3.2"/>
+<hole x="47.6" y="33.1" drill="3.2"/>
+<hole x="47.6" y="2" drill="3.2"/>
+<text x="46.9" y="30.8" size="1.27" layer="1" font="vector" ratio="15" rot="R270">C3MA Lightstick 20150714</text>
 </plain>
 <attributes>
@@
 <element name="U$1" library="lightstick" package="ESP8266" value="ESP8266" x="30.34" y="14.47" rot="MR270"/>
 <element name="U$2" library="lightstick" package="TO-263" value="LM2576S5,0" x="15.93" y="28.52" rot="R270"/>
-<element name="L1" library="Inductor-Fastron" package="PISR" value="L-EUPISR" x="28.61" y="14.23" rot="R90"/>
-<element name="C3" library="rcl" package="PANASONIC_D" value="100u" x="14.76" y="28.92" rot="MR270"/>
+<element name="L1" library="l-pwr-ind-lib" package="L12X12X7" value="L-PWRIND12X12X7" x="26.4" y="7.1" rot="R270"/>
+<element name="C3" library="rcl" package="PANASONIC_D" value="100u" x="7.74" y="5.88" rot="R90"/>
 <element name="C4" library="rcl" package="PANASONIC_F" value="470u" x="27.35" y="29.58"/>
 <element name="D1" library="diode" package="SMC" value="MBRS340T3" x="13.9" y="11.2" rot="R270"/>
-<element name="U$3" library="lightstick" package="AKL383-02" value="AKL383-02" x="3.9" y="22.7" rot="R270"/>
-<element name="U$4" library="lightstick" package="AKL383-02" value="AKL383-02" x="3.9" y="13" rot="R270"/>
+<element name="U$3" library="lightstick" package="AKL383-02" value="AKL383-02" x="3.1" y="25.4" rot="R270"/>
+<element name="U$4" library="lightstick" package="AKL383-02" value="AKL383-02" x="3" y="15.1" rot="R270"/>
 <element name="JP4" library="pinhead" package="1X01" value="" x="22.4" y="21.4"/>
 </elements>
@@
 <contactref element="U$2" pad="VIN"/>
 <contactref element="C3" pad="+"/>
-<wire x1="12.5264" y1="19.4464" x2="12.5264" y2="20.2015" width="0.4064" layer="1"/>
-<wire x1="14.76" y1="26.52" x2="10.39" y2="26.52" width="0.6096" layer="16"/>
 <contactref element="U$3" pad="PAD1"/>
 <contactref element="U$4" pad="PAD1"/>
-<wire x1="3.9" y1="14.905" x2="7.985" y2="14.905" width="1.6764" layer="16"/>
-<wire x1="10.39" y1="26.52" x2="8.475" y2="24.605" width="0.6096" layer="16"/>
-<wire x1="8.475" y1="24.605" x2="5.595" y2="24.605" width="0.6096" layer="16"/>
-<wire x1="3.9" y1="24.605" x2="5.595" y2="24.605" width="1.6764" layer="16"/>
-<via x="9.99" y="17.51" extent="1-16" drill="1" diameter="1.778"/>
-<wire x1="12.5264" y1="19.4464" x2="10.59" y2="17.51" width="1.27" layer="1"/>
-<wire x1="10.59" y1="17.51" x2="9.99" y2="17.51" width="1.27" layer="1"/>
-<wire x1="5.595" y1="24.605" x2="9.99" y2="20.21" width="1.6764" layer="16"/>
-<wire x1="9.99" y1="20.21" x2="9.99" y2="17.51" width="1.6764" layer="16"/>
-<wire x1="9.99" y1="17.51" x2="9.99" y2="16.91" width="1.6764" layer="16"/>
-<wire x1="9.99" y1="16.91" x2="7.985" y2="14.905" width="1.6764" layer="16"/>
+<wire x1="9.3299" y1="17.005" x2="7.74" y2="17.005" width="1.4224" layer="1"/>
+<wire x1="7.74" y1="17.005" x2="3" y2="17.005" width="1.4224" layer="1"/>
+<wire x1="9.7985" y1="20.2015" x2="8.7" y2="21.3" width="1.4224" layer="1"/>
+<wire x1="8.7" y1="21.3" x2="3.1" y2="27.305" width="1.4224" layer="1"/>
+<wire x1="7.74" y1="8.28" x2="7.74" y2="17.005" width="1.4224" layer="1"/>
+<wire x1="12.5264" y1="20.2015" x2="9.7985" y2="20.2015" width="1.27" layer="1"/>
+<wire x1="9.3299" y1="17.005" x2="9.3299" y2="20.2015" width="1.4224" layer="1"/>
+<wire x1="9.3299" y1="20.2015" x2="9.7985" y2="20.2015" width="1.4224" layer="1"/>
 </signal>
 <signal name="+5V">
@@
 <contactref element="C1" pad="1"/>
 <contactref element="U1" pad="3"/>
-<contactref element="L1" pad="2"/>
+<contactref element="L1" pad="P$2"/>
 <contactref element="U$2" pad="FEEDBACK"/>
 <contactref element="C4" pad="+"/>
 <via x="19.5" y="14.5" extent="1-16" drill="1" diameter="1.778"/>
-<wire x1="28.24" y1="22.4" x2="28.24" y2="27.22" width="1.6764" layer="1"/>
 <wire x1="28.24" y1="27.22" x2="28.54" y2="27.22" width="1.6764" layer="1"/>
 <wire x1="28.54" y1="27.22" x2="30.9" y2="29.58" width="1.6764" layer="1"/>
-<wire x1="28.6" y1="22.02" x2="28.61" y2="22.03" width="1.6764" layer="1"/>
 <wire x1="28.54" y1="13.4962" x2="28.0762" y2="13.96" width="0.6096" layer="16"/>
 <wire x1="28.0762" y1="13.96" x2="23.75" y2="13.96" width="0.6096" layer="16"/>
 <wire x1="23.75" y1="13.96" x2="20.04" y2="13.96" width="0.6096" layer="16"/>
 <wire x1="20.04" y1="13.96" x2="19.5" y2="14.5" width="0.6096" layer="16"/>
-<wire x1="28.24" y1="22.4" x2="28.61" y2="22.03" width="0.6096" layer="1"/>
 <wire x1="19.5" y1="14.5" x2="17.6318" y2="16.3682" width="0.6096" layer="1"/>
 <wire x1="17.6318" y1="16.3682" x2="17.6318" y2="20.2015" width="0.6096" layer="1"/>
-<wire x1="28.24" y1="22.4" x2="20.34" y2="14.5" width="0.6096" layer="1"/>
-<wire x1="20.34" y1="14.5" x2="19.5" y2="14.5" width="0.6096" layer="1"/>
 <wire x1="34.8" y1="31.63" x2="32.75" y2="29.58" width="1.27" layer="1"/>
 <wire x1="32.75" y1="29.58" x2="30.9" y2="29.58" width="1.27" layer="1"/>
+<wire x1="31.48" y1="7.1" x2="28.24" y2="10.34" width="1.6764" layer="1"/>
+<wire x1="28.24" y1="10.34" x2="28.24" y2="14.5" width="1.6764" layer="1"/>
+<wire x1="28.24" y1="14.5" x2="28.24" y2="27.22" width="1.6764" layer="1"/>
+<wire x1="19.5" y1="14.5" x2="28.24" y2="14.5" width="0.6096" layer="1"/>
 </signal>
 <signal name="RX">
@@
 <signal name="N$1">
 <contactref element="U$2" pad="OUTPUT"/>
-<contactref element="L1" pad="1"/>
+<contactref element="L1" pad="P$1"/>
 <wire x1="14.2282" y1="20.2015" x2="14.22" y2="20.1933" width="0.4064" layer="1"/>
-<wire x1="21.91" y1="6.43" x2="28.61" y2="6.43" width="1.6764" layer="1"/>
 <contactref element="D1" pad="C"/>
-<wire x1="21.91" y1="6.43" x2="13.9" y2="14.44" width="1.6764" layer="1"/>
-<wire x1="13.9" y1="14.44" x2="13.9" y2="14.9" width="1.6764" layer="1"/>
 <wire x1="14.2282" y1="20.2015" x2="14.2282" y2="14.9" width="1.6764" layer="1"/>
 <wire x1="14.2282" y1="14.9" x2="13.9" y2="14.9" width="1.6764" layer="1"/>
+<wire x1="14.2282" y1="14.9" x2="21.32" y2="7.1" width="1.6764" layer="1"/>
 </signal>
 <signal name="N$3">
@@
 </signal>
 </signals>
-<errors>
-</errors>
 </board>
 </drawing>

Commit message: PCB designed improved, minor changes
Parts:
- added JP5: (no value), pinhead:1X01
- L1: device l-pwr-ind-lib:L12X12X7 -> l-pwr-ind:L12X12X7
- moved C3 2.60 mm to (5.38, 6.96), turned to 0 degrees
- moved JP4 2.25 mm to (23.6, 23.3)
- moved L1 1.00 mm to (25.8, 7.90)
Connections:
- net GND: now also JP5.1
Routing:
- net +5V: track 54.5 -> 67.7 mm
- net N$1: track 16.2 -> 22.0 mm
- net +12V: track 31.2 -> 32.5 mm
Other:
- board text added: "C3MA Lightstick 20150717"
- board text removed: "C3MA Lightstick 20150714"
Changed lines of the file:
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@@
 <layer number="14" name="Route14" color="1" fill="6" visible="no" active="no"/>
 <layer number="15" name="Route15" color="4" fill="6" visible="no" active="no"/>
-<layer number="16" name="Bottom" color="1" fill="1" visible="yes" active="yes"/>
+<layer number="16" name="Bottom" color="1" fill="1" visible="no" active="yes"/>
 <layer number="17" name="Pads" color="2" fill="1" visible="yes" active="yes"/>
 <layer number="18" name="Vias" color="2" fill="1" visible="yes" active="yes"/>
-<layer number="19" name="Unrouted" color="6" fill="1" visible="yes" active="yes"/>
+<layer number="19" name="Unrouted" color="6" fill="1" visible="no" active="yes"/>
 <layer number="20" name="Dimension" color="15" fill="1" visible="yes" active="yes"/>
-<layer number="21" name="tPlace" color="7" fill="1" visible="yes" active="yes"/>
-<layer number="22" name="bPlace" color="7" fill="1" visible="yes" active="yes"/>
-<layer number="23" name="tOrigins" color="15" fill="1" visible="yes" active="yes"/>
-<layer number="24" name="bOrigins" color="15" fill="1" visible="yes" active="yes"/>
-<layer number="25" name="tNames" color="7" fill="1" visible="yes" active="yes"/>
-<layer number="26" name="bNames" color="7" fill="1" visible="yes" active="yes"/>
-<layer number="27" name="tValues" color="7" fill="1" visible="yes" active="yes"/>
-<layer number="28" name="bValues" color="7" fill="1" visible="yes" active="yes"/>
+<layer number="21" name="tPlace" color="7" fill="1" visible="no" active="yes"/>
+<layer number="22" name="bPlace" color="7" fill="1" visible="no" active="yes"/>
+<layer number="23" name="tOrigins" color="15" fill="1" visible="no" active="yes"/>
+<layer number="24" name="bOrigins" color="15" fill="1" visible="no" active="yes"/>
+<layer number="25" name="tNames" color="7" fill="1" visible="no" active="yes"/>
+<layer number="26" name="bNames" color="7" fill="1" visible="no" active="yes"/>
+<layer number="27" name="tValues" color="7" fill="1" visible="no" active="yes"/>
+<layer number="28" name="bValues" color="7" fill="1" visible="no" active="yes"/>
 <layer number="29" name="tStop" color="7" fill="3" visible="no" active="yes"/>
 <layer number="30" name="bStop" color="7" fill="6" visible="no" active="yes"/>
@@
 <layer number="37" name="tTest" color="7" fill="1" visible="no" active="yes"/>
 <layer number="38" name="bTest" color="7" fill="1" visible="no" active="yes"/>
-<layer number="39" name="tKeepout" color="4" fill="11" visible="yes" active="yes"/>
-<layer number="40" name="bKeepout" color="1" fill="11" visible="yes" active="yes"/>
-<layer number="41" name="tRestrict" color="4" fill="10" visible="yes" active="yes"/>
-<layer number="42" name="bRestrict" color="1" fill="10" visible="yes" active="yes"/>
-<layer number="43" name="vRestrict" color="2" fill="10" visible="yes" active="yes"/>
+<layer number="39" name="tKeepout" color="4" fill="11" visible="no" active="yes"/>
+<layer number="40" name="bKeepout" color="1" fill="11" visible="no" active="yes"/>
+<layer number="41" name="tRestrict" color="4" fill="10" visible="no" active="yes"/>
+<layer number="42" name="bRestrict" color="1" fill="10" visible="no" active="yes"/>
+<layer number="43" name="vRestrict" color="2" fill="10" visible="no" active="yes"/>
 <layer number="44" name="Drills" color="7" fill="1" visible="no" active="yes"/>
-<layer number="45" name="Holes" color="7" fill="1" visible="yes" active="yes"/>
+<layer number="45" name="Holes" color="7" fill="1" visible="no" active="yes"/>
 <layer number="46" name="Milling" color="3" fill="1" visible="no" active="yes"/>
 <layer number="47" name="Measures" color="7" fill="1" visible="no" active="yes"/>
-<layer number="48" name="Document" color="7" fill="1" visible="yes" active="yes"/>
-<layer number="49" name="Reference" color="7" fill="1" visible="yes" active="yes"/>
-<layer number="51" name="tDocu" color="7" fill="1" visible="yes" active="yes"/>
-<layer number="52" name="bDocu" color="7" fill="1" visible="yes" active="yes"/>
+<layer number="48" name="Document" color="7" fill="1" visible="no" active="yes"/>
+<layer number="49" name="Reference" color="7" fill="1" visible="no" active="yes"/>
+<layer number="51" name="tDocu" color="7" fill="1" visible="no" active="yes"/>
+<layer number="52" name="bDocu" color="7" fill="1" visible="no" active="yes"/>
 <layer number="91" name="Nets" color="2" fill="1" visible="no" active="no"/>
 <layer number="92" name="Busses" color="1" fill="1" visible="no" active="no"/>
@@
 <hole x="47.6" y="33.1" drill="3.2"/>
 <hole x="47.6" y="2" drill="3.2"/>
-<text x="46.9" y="30.8" size="1.27" layer="1" font="vector" ratio="15" rot="R270">C3MA Lightstick 20150714</text>
+<text x="46.9" y="30.8" size="1.27" layer="1" font="vector" ratio="15" rot="R270">C3MA Lightstick 20150717</text>
+<text x="48.1" y="30.5" size="1.27" layer="16" font="vector" ratio="15" rot="MR270">C3MA Lightstick 20150717</text>
 </plain>
 <attributes>
@@
 <element name="U$1" library="lightstick" package="ESP8266" value="ESP8266" x="30.34" y="14.47" rot="MR270"/>
 <element name="U$2" library="lightstick" package="TO-263" value="LM2576S5,0" x="15.93" y="28.52" rot="R270"/>
-<element name="L1" library="l-pwr-ind-lib" package="L12X12X7" value="L-PWRIND12X12X7" x="26.4" y="7.1" rot="R270"/>
-<element name="C3" library="rcl" package="PANASONIC_D" value="100u" x="7.74" y="5.88" rot="R90"/>
+<element name="L1" library="l-pwr-ind" package="L12X12X7" value="L-PWRIND12X12X7" x="25.8" y="7.9" rot="R270"/>
+<element name="C3" library="rcl" package="PANASONIC_D" value="100u" x="5.38" y="6.96"/>
 <element name="C4" library="rcl" package="PANASONIC_F" value="470u" x="27.35" y="29.58"/>
 <element name="D1" library="diode" package="SMC" value="MBRS340T3" x="13.9" y="11.2" rot="R270"/>
 <element name="U$3" library="lightstick" package="AKL383-02" value="AKL383-02" x="3.1" y="25.4" rot="R270"/>
 <element name="U$4" library="lightstick" package="AKL383-02" value="AKL383-02" x="3" y="15.1" rot="R270"/>
-<element name="JP4" library="pinhead" package="1X01" value="" x="22.4" y="21.4"/>
+<element name="JP4" library="pinhead" package="1X01" value="" x="23.6" y="23.3"/>
+<element name="JP5" library="pinhead" package="1X01" value="" x="33" y="24.6"/>
 </elements>
 <signals>
@@
 <contactref element="U$4" pad="PAD2"/>
 <contactref element="JP4" pad="1"/>
+<contactref element="JP5" pad="1"/>
 </signal>
 <signal name="+12V">
@@
 <wire x1="9.7985" y1="20.2015" x2="8.7" y2="21.3" width="1.4224" layer="1"/>
 <wire x1="8.7" y1="21.3" x2="3.1" y2="27.305" width="1.4224" layer="1"/>
-<wire x1="7.74" y1="8.28" x2="7.74" y2="17.005" width="1.4224" layer="1"/>
+<wire x1="7.78" y1="6.96" x2="7.74" y2="17.005" width="1.4224" layer="1"/>
 <wire x1="12.5264" y1="20.2015" x2="9.7985" y2="20.2015" width="1.27" layer="1"/>
 <wire x1="9.3299" y1="17.005" x2="9.3299" y2="20.2015" width="1.4224" layer="1"/>
@@
 <contactref element="U$2" pad="FEEDBACK"/>
 <contactref element="C4" pad="+"/>
-<via x="19.5" y="14.5" extent="1-16" drill="1" diameter="1.778"/>
-<wire x1="28.24" y1="27.22" x2="28.54" y2="27.22" width="1.6764" layer="1"/>
-<wire x1="28.54" y1="27.22" x2="30.9" y2="29.58" width="1.6764" layer="1"/>
 <wire x1="28.54" y1="13.4962" x2="28.0762" y2="13.96" width="0.6096" layer="16"/>
-<wire x1="28.0762" y1="13.96" x2="23.75" y2="13.96" width="0.6096" layer="16"/>
-<wire x1="23.75" y1="13.96" x2="20.04" y2="13.96" width="0.6096" layer="16"/>
-<wire x1="20.04" y1="13.96" x2="19.5" y2="14.5" width="0.6096" layer="16"/>
-<wire x1="19.5" y1="14.5" x2="17.6318" y2="16.3682" width="0.6096" layer="1"/>
-<wire x1="17.6318" y1="16.3682" x2="17.6318" y2="20.2015" width="0.6096" layer="1"/>
 <wire x1="34.8" y1="31.63" x2="32.75" y2="29.58" width="1.27" layer="1"/>
 <wire x1="32.75" y1="29.58" x2="30.9" y2="29.58" width="1.27" layer="1"/>
-<wire x1="31.48" y1="7.1" x2="28.24" y2="10.34" width="1.6764" layer="1"/>
-<wire x1="28.24" y1="10.34" x2="28.24" y2="14.5" width="1.6764" layer="1"/>
-<wire x1="28.24" y1="14.5" x2="28.24" y2="27.22" width="1.6764" layer="1"/>
-<wire x1="19.5" y1="14.5" x2="28.24" y2="14.5" width="0.6096" layer="1"/>
+<wire x1="17.6318" y1="20.2015" x2="17.5" y2="20.2015" width="0.4064" layer="1"/>
+<wire x1="17.5" y1="20.2015" x2="17.5" y2="13.9" width="0.4064" layer="1"/>
+<via x="17.5" y="13.9" extent="1-16" drill="1" diameter="1.778" shape="square"/>
+<wire x1="17.5" y1="13.9" x2="23.75" y2="13.9" width="0.4064" layer="16"/>
+<wire x1="23.75" y1="13.9" x2="23.75" y2="13.96" width="0.4064" layer="16"/>
+<wire x1="23.75" y1="13.96" x2="28.0762" y2="13.96" width="0.4064" layer="16"/>
+<wire x1="30.9" y1="29.58" x2="30.9" y2="22.1" width="1.6764" layer="1"/>
+<wire x1="30.9" y1="22.1" x2="29.1" y2="20.3" width="1.6764" layer="1"/>
+<wire x1="29.1" y1="20.3" x2="29.1" y2="8.1" width="1.6764" layer="1"/>
+<wire x1="29.1" y1="8.1" x2="29.3" y2="7.9" width="1.6764" layer="1"/>
+<wire x1="29.1" y1="8.1" x2="29.1" y2="17.5" width="0.4064" layer="1"/>
+<wire x1="29.1" y1="17.5" x2="20.3" y2="17.5" width="0.4064" layer="1"/>
+<wire x1="20.3" y1="17.5" x2="17.5" y2="13.9" width="0.4064" layer="1"/>
 </signal>
 <signal name="RX">
@@
 <wire x1="14.2282" y1="20.2015" x2="14.2282" y2="14.9" width="1.6764" layer="1"/>
 <wire x1="14.2282" y1="14.9" x2="13.9" y2="14.9" width="1.6764" layer="1"/>
-<wire x1="14.2282" y1="14.9" x2="21.32" y2="7.1" width="1.6764" layer="1"/>
+<wire x1="14.2282" y1="14.9" x2="14.2282" y2="12.7718" width="1.6764" layer="1"/>
+<wire x1="14.2282" y1="12.7718" x2="22.1" y2="4.9" width="1.6764" layer="1"/>
+<wire x1="22.1" y1="4.9" x2="22.1" y2="7.7" width="1.6764" layer="1"/>
+<wire x1="22.1" y1="7.7" x2="22.3" y2="7.9" width="1.6764" layer="1"/>
 </signal>
 <signal name="N$3">
