File: powersupply/lightstick.sch (EAGLE design)
At the start: 15 parts, among them U1 MCP1703AT-3302E/CB

Commit message: Board modified for new inductor, changed side of capacitor
Parts:
- L1: value L-EUPISR -> L-PWRIND12X12X7; device Inductor-Fastron:L-EUPISR -> l-pwr-ind-lib:L-PWRIND12X12X7
Connections:
- net +5V: now also L1.P$2; no longer L1.2
- net N$1: now also L1.P$1; no longer L1.1
Changed lines of the file:
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@@
 <?xml version="1.0" encoding="utf-8"?>
 <!DOCTYPE eagle SYSTEM "eagle.dtd">
-<eagle version="6.6.0">
+<eagle version="6.4">
 <drawing>
 <settings>
@@
 <part name="GND12" library="supply1" deviceset="GND" device=""/>
 <part name="P+7" library="supply1" deviceset="+12V" device=""/>
-<part name="L1" library="Inductor-Fastron" deviceset="L-EU" device="PISR"/>
+<part name="L1" library="l-pwr-ind-lib" deviceset="L-PWRIND12X12X7" device=""/>
 <part name="GND13" library="supply1" deviceset="GND" device=""/>
 <part name="C3" library="rcl" deviceset="CPOL-EU" device="D" value="100u"/>
@@
 </segment>
 <segment>
-<pinref part="L1" gate="G$1" pin="2"/>
+<pinref part="L1" gate="G$1" pin="P$2"/>
 <wire x1="154.94" y1="114.3" x2="157.48" y2="114.3" width="0.1524" layer="91"/>
 <pinref part="U$2" gate="A" pin="FEEDBACK"/>
@@
 <segment>
 <pinref part="U$2" gate="A" pin="OUTPUT"/>
-<pinref part="L1" gate="G$1" pin="1"/>
+<pinref part="L1" gate="G$1" pin="P$1"/>
 <wire x1="137.16" y1="114.3" x2="139.7" y2="114.3" width="0.1524" layer="91"/>
 <wire x1="139.7" y1="114.3" x2="144.78" y2="114.3" width="0.1524" layer="91"/>

Commit message: PCB designed improved, minor changes
Parts:
- added JP5: (no value), pinhead:PINHD-1X1
- L1: device l-pwr-ind-lib:L-PWRIND12X12X7 -> l-pwr-ind:L-PWRIND12X12X7
Connections:
- net GND: now also JP5.1
Changed lines of the file:
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@@
 <part name="GND12" library="supply1" deviceset="GND" device=""/>
 <part name="P+7" library="supply1" deviceset="+12V" device=""/>
-<part name="L1" library="l-pwr-ind-lib" deviceset="L-PWRIND12X12X7" device=""/>
+<part name="L1" library="l-pwr-ind" deviceset="L-PWRIND12X12X7" device=""/>
 <part name="GND13" library="supply1" deviceset="GND" device=""/>
 <part name="C3" library="rcl" deviceset="CPOL-EU" device="D" value="100u"/>
@@
 <part name="JP4" library="pinhead" deviceset="PINHD-1X1" device=""/>
 <part name="GND16" library="supply1" deviceset="GND" device=""/>
+<part name="JP5" library="pinhead" deviceset="PINHD-1X1" device=""/>
+<part name="GND17" library="supply1" deviceset="GND" device=""/>
 </parts>
 <sheets>
@@
 <instance part="JP4" gate="G$1" x="124.46" y="63.5"/>
 <instance part="GND16" gate="1" x="111.76" y="55.88"/>
+<instance part="JP5" gate="G$1" x="137.16" y="63.5" rot="R180"/>
+<instance part="GND17" gate="1" x="147.32" y="55.88"/>
 </instances>
 <busses>
@@
 <wire x1="111.76" y1="63.5" x2="111.76" y2="58.42" width="0.1524" layer="91" style="longdash"/>
 </segment>
+<segment>
+<pinref part="GND17" gate="1" pin="GND"/>
+<wire x1="139.7" y1="63.5" x2="147.32" y2="63.5" width="0.1524" layer="91"/>
+<wire x1="147.32" y1="63.5" x2="147.32" y2="58.42" width="0.1524" layer="91"/>
+<pinref part="JP5" gate="G$1" pin="1"/>
+</segment>
 </net>
